File: Hardware/automata.sch (KiCad schematic (older format))
At the start: 1 part, among them U1 MSP430G2553IN20

Commit message: Started developing schematic and circuit board.
Parts:
- added C1: 0.1uF, ~, symbol C
- added P1: PORT 1, ~, symbol CONN_8
- added P2: PORT 2, ~, symbol CONN_8
- added Q1: PN2222A, ~, symbol NPN
- added R1: 47k, ~, symbol R
Connections:
- net VCC: now reaches U1.1 (DVCC)
- net VCC: now also C1.1, R1.1
- net P2.2: now reaches U1.10 (P2.2/TA1.1)
- net P2.2: now also P2.3 (P3)
- net P2.3: now reaches U1.11 (P2.3/TA1.0)
- net P2.3: now also P2.4 (P4)
- net P2.4: now reaches U1.12 (P2.4/TA1.2)
- net P2.4: now also P2.5 (P5)
- net P2.5: now reaches U1.13 (P2.5/TA1.2)
- net P2.5: now also P2.6 (P6)
- net P1.6: now reaches U1.14 (P1.6/TA0.1/UCB0SOMI/UCB0SCL/A6/CA6/TDI/TCLK)
- net P1.6: now also P1.7 (P7)
- net P1.7: now reaches U1.15 (P1.7/CAOUT/UCB0SIMO/UCB0SDA/A7/CA7/TDO/TDI)
- net P1.7: now also P1.8 (P8)
- net RST: now reaches U1.16 (~RST~/NMI/SBWTDIO)
- net RST: now also R1.2
- net TEST: now reaches U1.17 (TEST/SBWTCK)
- net P2.7: now reaches U1.18 (XOUT/P2.7)
- net P2.7: now also P2.8 (P8)
- net P2.6: now reaches U1.19 (XIN/P2.6/TA0.1)
- net P2.6: now also P2.7 (P7)
- net P1.0: now reaches U1.2 (P1.0/TA0CLK/ACLK/A0/CA0)
- net P1.0: now also P1.1 (P1), Q1.2 (B)
- net GND: now reaches U1.20 (DVSS)
- net GND: now also C1.2
- net P1.1: now reaches U1.3 (P1.1/TA0.0/UCA0RXD/UCA0SOMI/A1/CA1)
- net P1.1: now also P1.2 (P2)
- net P1.2: now reaches U1.4 (P1.2/TA0.1/UCA0TXD/UCA0SIMO/A2/CA2)
- net P1.2: now also P1.3 (P3)
- net P1.3: now reaches U1.5 (P1.3/ADC10CLK/CAOUT/VREF-/VEREF-/A3/CA3)
- net P1.3: now also P1.4 (P4)
- net P1.4: now reaches U1.6 (P1.4/SMCLK/UCB0STE/UCA0CLK/VREF+/VEREF+/A4/CA4/TCK)
- net P1.4: now also P1.5 (P5)
- net P1.5: now reaches U1.7 (P1.5/TA0.0/UCB0CLK/UCA0STE/A5/CA5/TMS)
- net P1.5: now also P1.6 (P6)
- net P2.0: now reaches U1.8 (P2.0/TA1.0)
- net P2.0: now also P2.1 (P1)
- net P2.1: now reaches U1.9 (P2.1/TA1.1)
- net P2.1: now also P2.2 (P2)
- new net P1.0_COL: Q1.3 (C)
- new net P1.0_EMIT: Q1.1 (E)
Other:
- moved on the sheet: U1
Changed lines of the file:
@@
 LIBS:valves
 LIBS:embedded-microcontrollers
+LIBS:myparts
+LIBS:automata-cache
 EELAYER 27 0
 EELAYER END
@@
 Sheet 1 1
 Title ""
-Date "19 jan 2014"
+Date "15 apr 2014"
 Rev ""
 Comp ""
@@
 L MSP430G2553IN20 U1
 U 1 1 52DC27FD
-P 5800 3600
-F 0 "U1" H 8250 3700 60  0000 C CNN
-F 1 "MSP430G2553IN20" H 7100 2300 60  0000 C CNN
-F 2 "~" H 5800 3600 60  0000 C CNN
-F 3 "~" H 5800 3600 60  0000 C CNN
-	1    5800 3600
+P 4200 2900
+F 0 "U1" H 6650 3000 60  0000 C CNN
+F 1 "MSP430G2553IN20" H 5500 1600 60  0000 C CNN
+F 2 "~" H 4200 2900 60  0000 C CNN
+F 3 "~" H 4200 2900 60  0000 C CNN
+	1    4200 2900
 	1    0    0    -1
 $EndComp
+$Comp
+L VCC #PWR2
+U 1 1 534C74B0
+P 5500 2250
+F 0 "#PWR2" H 5500 2350 30  0001 C CNN
+F 1 "VCC" H 5500 2350 30  0000 C CNN
+F 2 "" H 5500 2250 60  0000 C CNN
+F 3 "" H 5500 2250 60  0000 C CNN
+	1    5500 2250
+	1    0    0    -1
+$EndComp
+$Comp
+L GND #PWR3
+U 1 1 534C74BF
+P 5500 5350
+F 0 "#PWR3" H 5500 5350 30  0001 C CNN
+F 1 "GND" H 5500 5280 30  0001 C CNN
+F 2 "" H 5500 5350 60  0000 C CNN
+F 3 "" H 5500 5350 60  0000 C CNN
+	1    5500 5350
+	1    0    0    -1
+$EndComp
+$Comp
+L R R1
+U 1 1 534C7525
+P 3400 4100
+F 0 "R1" V 3480 4100 40  0000 C CNN
+F 1 "47k" V 3407 4101 40  0000 C CNN
+F 2 "~" V 3330 4100 30  0000 C CNN
+F 3 "~" H 3400 4100 30  0000 C CNN
+	1    3400 4100
+	0    -1   -1   0
+$EndComp
+$Comp
+L VCC #PWR1
+U 1 1 534C756E
+P 3050 4100
+F 0 "#PWR1" H 3050 4200 30  0001 C CNN
+F 1 "VCC" V 3050 4200 30  0000 C CNN
+F 2 "" H 3050 4100 60  0000 C CNN
+F 3 "" H 3050 4100 60  0000 C CNN
+	1    3050 4100
+	0    -1   -1   0
+$EndComp
+$Comp
+L NPN Q1
+U 1 1 534C765B
+P 3650 3000
+F 0 "Q1" H 3650 2850 50  0000 R CNN
+F 1 "PN2222A" H 3650 3150 50  0000 R CNN
+F 2 "~" H 3650 3000 60  0000 C CNN
+F 3 "~" H 3650 3000 60  0000 C CNN
+	1    3650 3000
+	0    -1   -1   0
+$EndComp
+$Comp
+L C C1
+U 1 1 534C7858
+P 5700 2400
+F 0 "C1" H 5700 2500 40  0000 L CNN
+F 1 "0.1uF" H 5706 2315 40  0000 L CNN
+F 2 "~" H 5738 2250 30  0000 C CNN
+F 3 "~" H 5700 2400 60  0000 C CNN
+	1    5700 2400
+	0    -1   -1   0
+$EndComp
+$Comp
+L GND #PWR4
+U 1 1 534C788C
+P 6150 2400
+F 0 "#PWR4" H 6150 2400 30  0001 C CNN
+F 1 "GND" H 6150 2330 30  0001 C CNN
+F 2 "" H 6150 2400 60  0000 C CNN
+F 3 "" H 6150 2400 60  0000 C CNN
+	1    6150 2400
+	0    -1   -1   0
+$EndComp
+$Comp
+L CONN_8 P1
+U 1 1 534C8646
+P 2050 3700
+F 0 "P1" V 2000 3700 60  0000 C CNN
+F 1 "PORT 1" V 2100 3700 60  0000 C CNN
+F 2 "~" H 2050 3700 60  0000 C CNN
+F 3 "~" H 2050 3700 60  0000 C CNN
+	1    2050 3700
+	-1   0    0    1
+$EndComp
+Wire Wire Line
+	5500 5350 5500 4950
+Wire Wire Line
+	5500 2600 5500 2250
+Wire Wire Line
+	3900 4100 3650 4100
+Wire Wire Line
+	3900 3200 3650 3200
+Wire Wire Line
+	5900 2400 6150 2400
+Wire Wire Line
+	3150 4100 3050 4100
+Connection ~ 5500 2400
+Wire Wire Line
+	3850 2900 3850 2750
+Wire Wire Line
+	3450 2900 3450 2750
+Wire Wire Line
+	3900 3300 3650 3300
+Wire Wire Line
+	3900 3400 3650 3400
+Wire Wire Line
+	3900 3500 3650 3500
+Wire Wire Line
+	3900 3600 3650 3600
+Wire Wire Line
+	3900 3700 3650 3700
+Wire Wire Line
+	3900 3800 3650 3800
+Wire Wire Line
+	3900 3900 3650 3900
+Wire Wire Line
+	3900 4200 3000 4200
+Wire Wire Line
+	3900 4400 3650 4400
+Wire Wire Line
+	3900 4500 3650 4500
+Text Label 3650 4500 0    60   ~ 0
+P2.7
+Text Label 3650 4400 0    60   ~ 0
+P2.6
+Text Label 3000 4200 0    60   ~ 0
+TEST
+Wire Wire Line
+	3650 4100 3650 4000
+Wire Wire Line
+	3650 4000 3000 4000
+Text Label 3000 4000 0    60   ~ 0
+RST
+Text Label 3650 3900 0    60   ~ 0
+P1.7
+Text Label 3650 3800 0    60   ~ 0
+P1.6
+Text Label 3650 3700 0    60   ~ 0
+P1.5
+Text Label 3650 3600 0    60   ~ 0
+P1.4
+Text Label 3650 3500 0    60   ~ 0
+P1.3
+Text Label 3650 3400 0    60   ~ 0
+P1.2
+Text Label 3650 3300 0    60   ~ 0
+P1.1
+Text Label 3650 3200 0    60   ~ 0
+P1.0
+Text Label 3450 2750 1    60   ~ 0
+P1.0_COL
+Text Label 3850 2750 1    60   ~ 0
+P1.0_EMIT
+Text Label 2400 4050 0    60   ~ 0
+P1.0
+Text Label 2400 3950 0    60   ~ 0
+P1.1
+Text Label 2400 3850 0    60   ~ 0
+P1.2
+Text Label 2400 3750 0    60   ~ 0
+P1.3
+Text Label 2400 3650 0    60   ~ 0
+P1.4
+Text Label 2400 3550 0    60   ~ 0
+P1.5
+Text Label 2400 3450 0    60   ~ 0
+P1.6
+Text Label 2400 3350 0    60   ~ 0
+P1.7
+$Comp
+L CONN_8 P2
+U 1 1 534C8B6F
+P 2050 2800
+F 0 "P2" V 2000 2800 60  0000 C CNN
+F 1 "PORT 2" V 2100 2800 60  0000 C CNN
+F 2 "~" H 2050 2800 60  0000 C CNN
+F 3 "~" H 2050 2800 60  0000 C CNN
+	1    2050 2800
+	-1   0    0    1
+$EndComp
+Text Label 7000 4550 0    60   ~ 0
+P2.5
+Text Label 7000 4450 0    60   ~ 0
+P2.4
+Text Label 7000 4350 0    60   ~ 0
+P2.3
+Text Label 7000 4250 0    60   ~ 0
+P2.2
+Text Label 7000 4150 0    60   ~ 0
+P2.1
+Text Label 7000 4050 0    60   ~ 0
+P2.0
+Text Label 2400 3150 0    60   ~ 0
+P2.0
+Text Label 2400 3050 0    60   ~ 0
+P2.1
+Text Label 2400 2950 0    60   ~ 0
+P2.2
+Text Label 2400 2850 0    60   ~ 0
+P2.3
+Text Label 2400 2750 0    60   ~ 0
+P2.4
+Text Label 2400 2650 0    60   ~ 0
+P2.5
+Text Label 2400 2550 0    60   ~ 0
+P2.6
+Text Label 2400 2450 0    60   ~ 0
+P2.7
 $EndSCHEMATC
